File: Hardware/SparkFun ESP32 Thing Plus C.sch (EAGLE design)
At the start: 56 parts, among them J3 QWIIC_RIGHT_ANGLE, J6 microSD, Q2 MBT3904DW1T1, Q3 20V/4.2A/52mΩ/1.4W, U1 MCP73831, U2 ESP-WROOM-32NARROW, U3 AP2112K-3.3, U4 MAX17048, U5 AP2112K-3.3, U6 THINGPLUS_LOGICAL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

Commit message: Update file names
Other:
- note removed: "Add silk to allow for U.FL or trace antenna"
- note removed: "Rotate microSD"
Changed lines of the file:
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@@
 <text x="299.72" y="177.8" size="2.54" layer="94" font="vector" align="center">RGB Status LED</text>
 <text x="236.22" y="48.26" size="2.54" layer="94" font="vector" align="center">microSD Connector</text>
-<text x="449.58" y="132.08" size="1.27" layer="91">Add silk to allow for U.FL or trace antenna</text>
 <text x="226.06" y="129.54" size="1.27" layer="97" align="center">IO15: Has builtin pullup at POR.</text>
 <text x="226.06" y="134.62" size="1.27" layer="97" align="center">IO5: Has builtin pullup at POR.</text>
-<text x="449.58" y="129.54" size="1.778" layer="91">Rotate microSD</text>
 </plain>
 <instances>
